File: pcb/lithe-pcb.kicad_pcb (KiCad board)
At the start: 2 copper layers, 63.5 x 44.5 mm, 34 parts, among them J1 BUTTONS[8-9], J2 BUTTONS[0-3], J3 USB_B, J4 BUTTONS[4-7], J5 JOYSTICK, J6 TAG CONNECT, SW1 RESET, U1 MIC5504-3.3YM5, U2 ATSAMD21G18A-A, Y1 32.768KHz

Commit message: [pcb] Annoate parts with DigiKey P/Ns and add BOM.
Parts:
- R3, R4: value 400 -> 390
