File: pcb/lithe-pcb.sch (KiCad schematic (older format))
At the start: 34 parts, among them J1 BUTTONS[8-9], J2 BUTTONS[0-3], J3 USB_B, J4 BUTTONS[4-7], J5 JOYSTICK, J6 TAG CONNECT, SW1 RESET, U1 MIC5504-3.3YM5, U2 ATSAMD21G18A-A, Y1 32.768KHz

Commit message: [pcb] Annoate parts with DigiKey P/Ns and add BOM.
Parts:
- C1, C2, C8: DIGI_PN (none) -> 1276-6524-2-ND
- C3, C4: DIGI_PN (none) -> 311-2077-1-ND
- C5: DIGI_PN (none) -> 490-3298-1-ND
- C6, C7: DIGI_PN (none) -> 445-1239-1-ND
- D1: DIGI_PN (none) -> CLMVC-FKA-CL1D1L71BB7C3C3TR-ND
- J1: DIGI_PN (none) -> 277-5738-ND
- J2, J4: DIGI_PN (none) -> 277-5759-ND
- J5: DIGI_PN (none) -> 277-5752-ND
- R1: DIGI_PN (none) -> YAG2307TR-ND
- R2: DIGI_PN (none) -> 311-620LRTR-ND
- R3, R4: value 400 -> 390; DIGI_PN (none) -> 311-390LRTR-ND
- R5: DIGI_PN (none) -> 311-1.00KLRTR-ND
- R6, R7, R8, R9: DIGI_PN (none) -> 311-0.0JRTR-ND
- SW1: DIGI_PN (none) -> CKN12311-2-ND
- U1: DIGI_PN (none) -> MIC5504-3.3YM5-T5TR-ND
- U2: DIGI_PN (none) -> ATSAMD21G18A-AU-ND
- Y1: DIGI_PN (none) -> 2195-CM7VT1ALOWESR32.768KHZ12.5PF20TAQCTR-ND
Changed lines of the file:
@@
 F 2 "Package_QFP:TQFP-48_7x7mm_P0.5mm" H 9750 1750 50  0001 C CNN
 F 3 "http://ww1.microchip.com/downloads/en/DeviceDoc/SAM_D21_DA1_Family_Data%20Sheet_DS40001882E.pdf" H 8850 4600 50  0001 C CNN
+F 4 "ATSAMD21G18A-AU-ND" H 8850 3600 50  0001 C CNN "DIGI_PN"
 	1    8850 3600
 	1    0    0    -1
@@
 F 2 "Capacitor_SMD:C_0402_1005Metric" H 8350 1600 50  0001 C CNN
 F 3 "~" H 8350 1600 50  0001 C CNN
+F 4 "1276-6524-2-ND" H 8350 1600 50  0001 C CNN "DIGI_PN"
 	1    8350 1600
 	0    1    1    0
@@
 F 2 "Capacitor_SMD:C_0402_1005Metric" H 6600 2350 50  0001 C CNN
 F 3 "~" H 6600 2350 50  0001 C CNN
+F 4 "445-1239-1-ND" H 6600 2350 50  0001 C CNN "DIGI_PN"
 	1    6600 2350
 	1    0    0    -1
@@
 F 2 "Capacitor_SMD:C_0402_1005Metric" H 6950 2350 50  0001 C CNN
 F 3 "~" H 6950 2350 50  0001 C CNN
+F 4 "445-1239-1-ND" H 6950 2350 50  0001 C CNN "DIGI_PN"
 	1    6950 2350
 	1    0    0    -1
@@
 F 2 "Package_TO_SOT_SMD:SOT-23-5" H 2300 1050 50  0001 C CNN
 F 3 "http://ww1.microchip.com/downloads/en/DeviceDoc/MIC550X.pdf" H 2050 1700 50  0001 C CNN
+F 4 "MIC5504-3.3YM5-T5TR-ND" H 2300 1450 50  0001 C CNN "DIGI_PN"
 	1    2300 1450
 	1    0    0    -1
@@
 F 2 "Capacitor_SMD:C_0402_1005Metric" H 1150 1550 50  0001 C CNN
 F 3 "~" H 1150 1550 50  0001 C CNN
+F 4 "1276-6524-2-ND" H 1150 1550 50  0001 C CNN "DIGI_PN"
 	1    1150 1550
 	1    0    0    -1
@@
 F 2 "Capacitor_SMD:C_0402_1005Metric" H 2800 1550 50  0001 C CNN
 F 3 "~" H 2800 1550 50  0001 C CNN
+F 4 "1276-6524-2-ND" H 2800 1550 50  0001 C CNN "DIGI_PN"
 	1    2800 1550
 	1    0    0    -1
@@
 F 2 "Button_Switch_SMD:SW_SPST_EVQPE1" H 5100 6800 50  0001 C CNN
 F 3 "~" H 5100 6800 50  0001 C CNN
+F 4 "CKN12311-2-ND" H 5100 6600 50  0001 C CNN "DIGI_PN"
 	1    5100 6600
 	1    0    0    -1
@@
 F 2 "Capacitor_SMD:C_0603_1608Metric" H 5450 1500 50  0001 C CNN
 F 3 "~" H 5450 1500 50  0001 C CNN
+F 4 "490-3298-1-ND" H 5450 1500 50  0001 C CNN "DIGI_PN"
 	1    5450 1500
 	1    0    0    -1
@@
 F 2 "Capacitor_SMD:C_0402_1005Metric" H 4500 1500 50  0001 C CNN
 F 3 "~" H 4500 1500 50  0001 C CNN
+F 4 "311-2077-1-ND" H 4500 1500 50  0001 C CNN "DIGI_PN"
 	1    4500 1500
 	1    0    0    -1
@@
 F 2 "Capacitor_SMD:C_0402_1005Metric" H 5000 1500 50  0001 C CNN
 F 3 "~" H 5000 1500 50  0001 C CNN
+F 4 "311-2077-1-ND" H 5000 1500 50  0001 C CNN "DIGI_PN"
 	1    5000 1500
 	1    0    0    -1
@@
 F 2 "Resistor_SMD:R_0402_1005Metric" H 5450 3800 50  0001 C CNN
 F 3 "~" H 5450 3800 50  0001 C CNN
+F 4 "311-1.00KLRTR-ND" H 5450 3800 50  0001 C CNN "DIGI_PN"
 	1    5450 3800
 	1    0    0    -1
@@
 F 2 "Resistor_SMD:R_0402_1005Metric" H 1500 1550 50  0001 C CNN
 F 3 "~" H 1500 1550 50  0001 C CNN
+F 4 "YAG2307TR-ND" H 1500 1550 50  0001 C CNN "DIGI_PN"
 	1    1500 1550
 	1    0    0    -1
@@
 F 2 "LED_SMD:LED_Cree-PLCC4_2x2mm_CW" H 5100 5450 50  0001 C CNN
 F 3 "~" H 5100 5450 50  0001 C CNN
+F 4 "CLMVC-FKA-CL1D1L71BB7C3C3TR-ND" H 5100 5500 50  0001 C CNN "DIGI_PN"
 	1    5100 5500
 	1    0    0    -1
@@
 P 4700 5700
 F 0 "R4" V 4600 5750 50  0000 C CNN
-F 1 "400" V 4600 5600 50  0000 C CNN
+F 1 "390" V 4600 5600 50  0000 C CNN
 F 2 "Resistor_SMD:R_0402_1005Metric" H 4700 5700 50  0001 C CNN
 F 3 "~" H 4700 5700 50  0001 C CNN
+F 4 "311-390LRTR-ND" H 4700 5700 50  0001 C CNN "DIGI_PN"
 	1    4700 5700
 	0    1    1    0
@@
 P 4700 5500
 F 0 "R3" V 4600 5550 50  0000 C CNN
-F 1 "400" V 4600 5400 50  0000 C CNN
+F 1 "390" V 4600 5400 50  0000 C CNN
 F 2 "Resistor_SMD:R_0402_1005Metric" H 4700 5500 50  0001 C CNN
 F 3 "~" H 4700 5500 50  0001 C CNN
+F 4 "311-390LRTR-ND" H 4700 5500 50  0001 C CNN "DIGI_PN"
 	1    4700 5500
 	0    1    1    0
@@
 F 2 "Resistor_SMD:R_0402_1005Metric" H 4700 5300 50  0001 C CNN
 F 3 "~" H 4700 5300 50  0001 C CNN
+F 4 "311-620LRTR-ND" H 4700 5300 50  0001 C CNN "DIGI_PN"
 	1    4700 5300
 	0    1    1    0
@@
 F 2 "Crystal:Crystal_SMD_MicroCrystal_CC7V-T1A-2Pin_3.2x1.5mm_HandSoldering" H 6950 2050 50  0001 C CNN
 F 3 "~" H 6950 2050 50  0001 C CNN
+F 4 "2195-CM7VT1ALOWESR32.768KHZ12.5PF20TAQCTR-ND" H 6950 2050 50  0001 C CNN "DIGI_PN"
 	1    6950 2050
 	0    1    1    0
@@
 F 2 "Connector_Phoenix_MC:PhoenixContact_MCV_1,5_5-G-3.5_1x05_P3.50mm_Vertical" H 2950 6900 50  0001 C CNN
 F 3 "~" H 2950 6900 50  0001 C CNN
+F 4 "277-5752-ND" H 2950 6900 50  0001 C CNN "DIGI_PN"
 	1    2950 6900
 	1    0    0    -1
@@
 F 2 "Connector_Phoenix_MC:PhoenixContact_MCV_1,5_4-G-3.5_1x04_P3.50mm_Vertical" H 1900 6900 50  0001 C CNN
 F 3 "~" H 1900 6900 50  0001 C CNN
+F 4 "277-5738-ND" H 1900 6900 50  0001 C CNN "DIGI_PN"
 	1    1900 6900
 	1    0    0    -1
@@
 F 2 "Connector_Phoenix_MC:PhoenixContact_MCV_1,5_8-G-3.5_1x08_P3.50mm_Vertical" H 2950 5550 50  0001 C CNN
 F 3 "~" H 2950 5550 50  0001 C CNN
+F 4 "277-5759-ND" H 2950 5550 50  0001 C CNN "DIGI_PN"
 	1    2950 5550
 	1    0    0    -1
@@
 F 2 "Connector_Phoenix_MC:PhoenixContact_MCV_1,5_8-G-3.5_1x08_P3.50mm_Vertical" H 1950 5550 50  0001 C CNN
 F 3 "~" H 1950 5550 50  0001 C CNN
+F 4 "277-5759-ND" H 1950 5550 50  0001 C CNN "DIGI_PN"
 	1    1950 5550
 	1    0    0    -1
@@
 F 2 "Resistor_SMD:R_0402_1005Metric" H 7150 4500 50  0001 C CNN
 F 3 "~" H 7150 4500 50  0001 C CNN
+F 4 "311-0.0JRTR-ND" H 7150 4500 50  0001 C CNN "DIGI_PN"
 	1    7150 4500
 	1    0    0    -1
@@
 F 2 "Resistor_SMD:R_0402_1005Metric" H 6900 4500 50  0001 C CNN
 F 3 "~" H 6900 4500 50  0001 C CNN
+F 4 "311-0.0JRTR-ND" H 6900 4500 50  0001 C CNN "DIGI_PN"
 	1    6900 4500
 	1    0    0    -1
@@
 F 2 "Resistor_SMD:R_0402_1005Metric" H 6650 4500 50  0001 C CNN
 F 3 "~" H 6650 4500 50  0001 C CNN
+F 4 "311-0.0JRTR-ND" H 6650 4500 50  0001 C CNN "DIGI_PN"
 	1    6650 4500
 	1    0    0    -1
@@
 F 2 "Resistor_SMD:R_0402_1005Metric" H 6400 4500 50  0001 C CNN
 F 3 "~" H 6400 4500 50  0001 C CNN
+F 4 "311-0.0JRTR-ND" H 6400 4500 50  0001 C CNN "DIGI_PN"
 	1    6400 4500
 	1    0    0    -1
@@
 	6400 4300 8150 4300
 $Comp
-L power:GND #PWR?
+L power:GND #PWR0128
 U 1 1 600C7DC4
 P 6400 4700
-F 0 "#PWR?" H 6400 4450 50  0001 C CNN
+F 0 "#PWR0128" H 6400 4450 50  0001 C CNN
 F 1 "GND" H 6405 4527 50  0000 C CNN
 F 2 "" H 6400 4700 50  0001 C CNN
@@
 $EndComp
 $Comp
-L power:GND #PWR?
+L power:GND #PWR0129
 U 1 1 600C8928
 P 6650 4700
-F 0 "#PWR?" H 6650 4450 50  0001 C CNN
+F 0 "#PWR0129" H 6650 4450 50  0001 C CNN
 F 1 "GND" H 6655 4527 50  0000 C CNN
 F 2 "" H 6650 4700 50  0001 C CNN
@@
 $EndComp
 $Comp
-L power:GND #PWR?
+L power:GND #PWR0130
 U 1 1 600C8DB0
 P 6900 4700
-F 0 "#PWR?" H 6900 4450 50  0001 C CNN
+F 0 "#PWR0130" H 6900 4450 50  0001 C CNN
 F 1 "GND" H 6905 4527 50  0000 C CNN
 F 2 "" H 6900 4700 50  0001 C CNN
@@
 $EndComp
 $Comp
-L power:GND #PWR?
+L power:GND #PWR0131
 U 1 1 600C957C
 P 7150 4700
-F 0 "#PWR?" H 7150 4450 50  0001 C CNN
+F 0 "#PWR0131" H 7150 4450 50  0001 C CNN
 F 1 "GND" H 7155 4527 50  0000 C CNN
 F 2 "" H 7150 4700 50  0001 C CNN
